File: keyMatrix.sch (KiCad schematic (older format))
At the start: 150 parts

Commit message: commit
Parts:
- removed D? (x74): D, symbol Device:D
- removed SW? (x74): SW_Push, symbol Switch:SW_Push
- added D? (x79): D, symbol Device:D
- added SW? (x79): SW_Push, symbol Switch:SW_Push
Connections:
- net row0 is gone; now on net col0: D?.1 (K)
- net col0: now also D?.1 (K), D?.1 (K), D?.1 (K), D?.1 (K), D?.1 (K), D?.1 (K), D?.1 (K), D?.1 (K), D?.1 (K), D?.1 (K), D?.1 (K), D?.1 (K)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
- new net: D?.2 (A), SW?.1 (x79)
Other:
- moved on the sheet: D?, SW?
